Commit message: 增加可调控方向摄像头

File: src/patrol_robot_description/urdf/patrol_robot.urdf.xacro (robot description, xacro)
@@ -163,4 +163,58 @@
     <origin xyz="0 0 0.12" rpy="0 0 0"/>
   </joint>
+  <!--
+    两轴 RGB-D 云台：水平关节绕 Z 轴旋转，俯仰关节绕 Y 轴旋转。
+    真机可保留相同关节和控制话题，仅替换外参及舵机驱动。
+  -->
+  <link name="camera_pan_link">
+    <visual>
+      <geometry><cylinder radius="0.035" length="0.035"/></geometry>
+      <material name="sensor_gray"/>
+    </visual>
+    <collision>
+      <geometry><cylinder radius="0.035" length="0.035"/></geometry>
+    </collision>
+    <inertial>
+      <mass value="0.08"/>
+      <inertia ixx="0.00004" ixy="0" ixz="0" iyy="0.00004" iyz="0" izz="0.00005"/>
+    </inertial>
+  </link>
+  <joint name="camera_pan_joint" type="revolute">
+    <parent link="base_link"/>
+    <child link="camera_pan_link"/>
+    <origin xyz="0.22 0 0.255" rpy="0 0 0"/>
+    <axis xyz="0 0 1"/>
+    <limit lower="${-pi / 2.0}" upper="${pi / 2.0}" effort="2.0" velocity="1.2"/>
+    <dynamics damping="0.12" friction="0.03"/>
+  </joint>
+  <link name="camera_link">
+    <visual>
+      <geometry><box size="0.07 0.13 0.05"/></geometry>
+      <material name="sensor_gray"/>
+    </visual>
+    <collision>
+      <geometry><box size="0.07 0.13 0.05"/></geometry>
+    </collision>
+    <inertial>
+      <mass value="0.12"/>
+      <inertia ixx="0.00019" ixy="0" ixz="0" iyy="0.00007" iyz="0" izz="0.00022"/>
+    </inertial>
+  </link>
+  <joint name="camera_tilt_joint" type="revolute">
+    <parent link="camera_pan_link"/>
+    <child link="camera_link"/>
+    <origin xyz="0.02 0 0.035" rpy="0 0 0"/>
+    <axis xyz="0 1 0"/>
+    <!-- 物理关节正方向为向下；网页接口会转换为“向上为正”。 -->
+    <limit lower="-0.436332" upper="0.610865" effort="2.0" velocity="1.0"/>
+    <dynamics damping="0.10" friction="0.03"/>
+  </joint>
+  <!-- ROS REP-103 光学坐标系：+Z 向前、+X 向右、+Y 向下。 -->
+  <link name="camera_depth_optical_frame"/>
+  <joint name="camera_depth_optical_joint" type="fixed">
+    <parent link="camera_link"/>
+    <child link="camera_depth_optical_frame"/>
+    <origin xyz="0.036 0 0" rpy="${-pi / 2.0} 0 ${-pi / 2.0}"/>
+  </joint>
   <gazebo reference="base_link">
     <material>Gazebo/Blue</material>
@@ -203,4 +257,33 @@
     </sensor>
   </gazebo>
+  <gazebo reference="camera_pan_link">
+    <material>Gazebo/DarkGrey</material>
+  </gazebo>
+  <gazebo reference="camera_link">
+    <sensor name="rgbd_camera" type="rgbd_camera">
+      <topic>/camera</topic>
+      <gz_frame_id>camera_depth_optical_frame</gz_frame_id>
+      <update_rate>15</update_rate>
+      <always_on>true</always_on>
+      <visualize>false</visualize>
+      <camera>
+        <horizontal_fov>1.04719755</horizontal_fov>
+        <image>
+          <width>640</width>
+          <height>480</height>
+          <format>R8G8B8</format>
+        </image>
+        <clip>
+          <near>0.20</near>
+          <far>8.0</far>
+        </clip>
+        <noise>
+          <type>gaussian</type>
+          <mean>0.0</mean>
+          <stddev>0.002</stddev>
+        </noise>
+      </camera>
+    </sensor>
+  </gazebo>
   <gazebo>
     <plugin filename="gz-sim-diff-drive-system" name="gz::sim::systems::DiffDrive">
@@ -237,4 +320,20 @@
       <joint_name>left_wheel_joint</joint_name>
       <joint_name>right_wheel_joint</joint_name>
+      <joint_name>camera_pan_joint</joint_name>
+      <joint_name>camera_tilt_joint</joint_name>
+    </plugin>
+    <plugin filename="gz-sim-joint-position-controller-system" name="gz::sim::systems::JointPositionController">
+      <joint_name>camera_pan_joint</joint_name>
+      <topic>/camera/gimbal/pan/command</topic>
+      <initial_position>0.0</initial_position>
+      <use_velocity_commands>true</use_velocity_commands>
+      <cmd_max>1.2</cmd_max>
+    </plugin>
+    <plugin filename="gz-sim-joint-position-controller-system" name="gz::sim::systems::JointPositionController">
+      <joint_name>camera_tilt_joint</joint_name>
+      <topic>/camera/gimbal/tilt/command</topic>
+      <initial_position>0.0</initial_position>
+      <use_velocity_commands>true</use_velocity_commands>
+      <cmd_max>1.0</cmd_max>
     </plugin>
   </gazebo>

Commit message: 过渡点设置，健康监测

File: src/patrol_robot_description/urdf/patrol_robot.urdf.xacro (robot description, xacro)
@@ -1,4 +1,5 @@
 <?xml version="1.0"?>
 <robot xmlns:xacro="http://www.ros.org/wiki/xacro" name="patrol_robot">
+  <xacro:arg name="ground_truth_odometry" default="true"/>
   <!-- 将来适配真机时，优先修改下面这些尺寸和质量。 -->
   <xacro:property name="base_length" value="0.52"/>
@@ -217,7 +218,4 @@
     <origin xyz="0.036 0 0" rpy="${-pi / 2.0} 0 ${-pi / 2.0}"/>
   </joint>
-  <gazebo reference="base_link">
-    <material>Gazebo/Blue</material>
-  </gazebo>
   <gazebo reference="laser_link">
     <sensor name="lidar" type="gpu_lidar">
@@ -255,8 +253,15 @@
       <update_rate>50</update_rate>
       <always_on>true</always_on>
+      <angular_velocity>
+        <x><noise type="gaussian"><mean>0</mean><stddev>0.002</stddev><bias_mean>0.0002</bias_mean><bias_stddev>0.0001</bias_stddev></noise></x>
+        <y><noise type="gaussian"><mean>0</mean><stddev>0.002</stddev><bias_mean>0.0002</bias_mean><bias_stddev>0.0001</bias_stddev></noise></y>
+        <z><noise type="gaussian"><mean>0</mean><stddev>0.004</stddev><bias_mean>0.0005</bias_mean><bias_stddev>0.0002</bias_stddev></noise></z>
+      </angular_velocity>
+      <linear_acceleration>
+        <x><noise type="gaussian"><mean>0</mean><stddev>0.03</stddev><bias_mean>0.01</bias_mean><bias_stddev>0.005</bias_stddev></noise></x>
+        <y><noise type="gaussian"><mean>0</mean><stddev>0.03</stddev><bias_mean>0.01</bias_mean><bias_stddev>0.005</bias_stddev></noise></y>
+        <z><noise type="gaussian"><mean>0</mean><stddev>0.04</stddev><bias_mean>0.01</bias_mean><bias_stddev>0.005</bias_stddev></noise></z>
+      </linear_acceleration>
     </sensor>
-  </gazebo>
-  <gazebo reference="camera_pan_link">
-    <material>Gazebo/DarkGrey</material>
   </gazebo>
   <gazebo reference="camera_link">
@@ -264,5 +269,6 @@
       <topic>/camera</topic>
       <gz_frame_id>camera_depth_optical_frame</gz_frame_id>
-      <update_rate>15</update_rate>
+      <!-- 10 Hz 足以支撑室内低速避障，并给 Nav2 控制循环预留 CPU。 -->
+      <update_rate>10</update_rate>
       <always_on>true</always_on>
       <visualize>false</visualize>
@@ -302,18 +308,26 @@
       <max_angular_acceleration>1.8</max_angular_acceleration>
     </plugin>
-    <!--
-      3D 物理仿真会出现轮胎滑移。若用轮速积分发布 odom，物理车体上的
-      laser_link 会逐渐与 TF 中的机器人分离，激光点云便会在地图中形成
-      假墙。OdometryPublisher 直接使用 Gazebo 模型实际位姿，使导航、
-      机器人模型和激光传感器始终处于同一坐标位置。
-    -->
-    <plugin filename="gz-sim-odometry-publisher-system" name="gz::sim::systems::OdometryPublisher">
-      <odom_frame>odom</odom_frame>
-      <robot_base_frame>base_footprint</robot_base_frame>
-      <odom_topic>/odom</odom_topic>
-      <tf_topic>/tf</tf_topic>
-      <odom_publish_frequency>30</odom_publish_frequency>
-      <dimensions>2</dimensions>
-    </plugin>
+    <!-- Keep truth available for comparison, but let the default navigation
+         profile expose wheel slip and IMU drift through an EKF. -->
+    <xacro:if value="$(arg ground_truth_odometry)">
+      <plugin filename="gz-sim-odometry-publisher-system" name="gz::sim::systems::OdometryPublisher">
+        <odom_frame>odom</odom_frame>
+        <robot_base_frame>base_footprint</robot_base_frame>
+        <odom_topic>/odom</odom_topic>
+        <tf_topic>/tf</tf_topic>
+        <odom_publish_frequency>30</odom_publish_frequency>
+        <dimensions>2</dimensions>
+      </plugin>
+    </xacro:if>
+    <xacro:unless value="$(arg ground_truth_odometry)">
+      <plugin filename="gz-sim-odometry-publisher-system" name="gz::sim::systems::OdometryPublisher">
+        <odom_frame>ground_truth_odom</odom_frame>
+        <robot_base_frame>base_footprint</robot_base_frame>
+        <odom_topic>/ground_truth/odom</odom_topic>
+        <tf_topic>/ground_truth/tf</tf_topic>
+        <odom_publish_frequency>30</odom_publish_frequency>
+        <dimensions>2</dimensions>
+      </plugin>
+    </xacro:unless>
     <plugin filename="gz-sim-joint-state-publisher-system" name="gz::sim::systems::JointStatePublisher">
       <topic>/joint_states</topic>
